File: pcb/pybox3_010/pybox3_010.kicad_pcb (KiCad board)
At the start: 2 copper layers, 66 x 53.3 mm, 9 parts, among them SW1 SW_Push, SW2 SW_Push, SW3 RotaryEncoder_Switch, U1 RP2040-ZERO

Commit message: update
Parts:
- added HL1: MountingHole_3.2mm_M3, MountingHole:MountingHole_3.2mm_M3, F.Cu at (239.6, 88.9)
- added HL2: MountingHole_3.2mm_M3, MountingHole:MountingHole_3.2mm_M3, F.Cu at (187.3, 75.6)
- added HL3: MountingHole_3.2mm_M3, MountingHole:MountingHole_3.2mm_M3, F.Cu at (187.3, 102.2)
- U1: footprint RP2040-ZERO:MODULE_RP2040-ZERO -> RP2040-ZERO:MODULE_RP2040-ZERO_reduced
- moved G*** 0.64 mm to (228.0, 88.9)
- moved SW3 0.07 mm to (209.7, 86.4)
Routing:
- net Net-(BZ2-+): track 47.6 -> 41.0 mm
- net GND: track 147.5 -> 142.4 mm
- net Net-(U1-GP0): track 49.7 -> 48.8 mm
- added copper zone on B.Cu, net GND
- added copper zone on F.Cu, net GND
Other:
- board size 66 x 53.3 mm -> 65.5 x 53.3 mm

Commit message: FIXED: new pcb ready (3.0.1)
Routing:
- net VCC: track 50.4 -> 59.6 mm
- net GND: track 142.4 -> 138.5 mm
- net Net-(BZ1-+): track 41.0 -> 44.1 mm
- net Net-(U1-GP27): track 25.9 -> 24.7 mm
Other:
- board text added: "pybox v3.0.1 2025-03"
- board text removed: "pybox v3.0.0 2025-02"
